File: VoltAir.kicad_pcb (KiCad board)
At the start: 2 copper layers, 2 parts, among them J1 Conn_01x06_Pin, U1 ESP32-WROOM-32

Commit message: initial layout
Parts:
- added C1: 0.1u, Capacitor_SMD:C_0603_1608Metric, F.Cu at (128.2, 31.9)
- added C10: 1u, Capacitor_SMD:C_0603_1608Metric, F.Cu at (128.2, 36.9)
- added C11: C, Capacitor_THT:CP_Radial_D8.0mm_P5.00mm, F.Cu at (173.4, 78.3)
- added C12: C, Capacitor_THT:CP_Radial_D8.0mm_P5.00mm, F.Cu at (173.4, 67.2)
- added C13: C, Capacitor_THT:CP_Radial_D8.0mm_P5.00mm, F.Cu at (215.5, 83.1)
- added C14: C, Capacitor_THT:CP_Radial_D8.0mm_P5.00mm, F.Cu at (215.5, 72.0)
- added C2: 0.1u, Capacitor_SMD:C_0603_1608Metric, F.Cu at (120.4, 51.0)
- added C3: 0.1u, Capacitor_SMD:C_0603_1608Metric, F.Cu at (128.2, 34.4)
- added C4: 10u, Capacitor_Tantalum_SMD:CP_EIA-3216-18_Kemet-A_Pad1.58x1.35mm_HandSolder, F.Cu at (133.3, 37.3)
- added C5: 0.1u, Capacitor_SMD:C_0603_1608Metric, F.Cu at (120.4, 53.5)
- added C6: 0.1u, Capacitor_SMD:C_0603_1608Metric, F.Cu at (120.4, 56.0)
- added C7: 0.1u, Capacitor_SMD:C_0603_1608Metric, F.Cu at (120.4, 58.5)
- added C8: 10u, Capacitor_Tantalum_SMD:CP_EIA-3216-18_Kemet-A_Pad1.58x1.35mm_HandSolder, F.Cu at (129.3, 64.9)
- added C9: 10u, Capacitor_Tantalum_SMD:CP_EIA-3216-18_Kemet-A_Pad1.58x1.35mm_HandSolder, F.Cu at (129.3, 68.0)
- added D1: LED, LED_SMD:LED_0603_1608Metric, F.Cu at (134.3, 64.6)
- added D2: LED, LED_SMD:LED_0603_1608Metric, F.Cu at (138.3, 37.0)
- added J2: Conn_01x02, TestPoint:TestPoint_2Pads_Pitch5.08mm_Drill1.3mm, F.Cu at (219.5, 83.2)
- added J3: Conn_01x02, TestPoint:TestPoint_2Pads_Pitch5.08mm_Drill1.3mm, F.Cu at (219.5, 72.0)
- added J4: Conn_01x02, Connector_Molex:Molex_PicoBlade_53047-0210_1x02_P1.25mm_Vertical, F.Cu at (125.8, 80.5)
- added J5: Conn_01x02, TestPoint:TestPoint_2Pads_Pitch5.08mm_Drill1.3mm, F.Cu at (169.4, 78.2)
- added J6: Conn_01x02, TestPoint:TestPoint_2Pads_Pitch5.08mm_Drill1.3mm, F.Cu at (169.4, 67.0)
- added R1: 10k, Resistor_SMD:R_0603_1608Metric, F.Cu at (128.2, 39.4)
- added R10: 100R, Resistor_SMD:R_0603_1608Metric, F.Cu at (128.2, 41.9)
- added R11: 100R, Resistor_SMD:R_0603_1608Metric, F.Cu at (128.2, 44.5)
- added R12: 100R, Resistor_SMD:R_0603_1608Metric, F.Cu at (128.2, 47.0)
- added R13: 100R, Resistor_SMD:R_0603_1608Metric, F.Cu at (128.2, 49.5)
- added R14: 560R, Resistor_SMD:R_0603_1608Metric, F.Cu at (128.2, 52.0)
- added R2: 100R, Resistor_SMD:R_0603_1608Metric, F.Cu at (181.5, 92.4)
- added R3: 100R, Resistor_SMD:R_0603_1608Metric, F.Cu at (183.7, 92.4)
- added R4: 100R, Resistor_SMD:R_0603_1608Metric, F.Cu at (185.8, 92.4)
- added R5: 100R, Resistor_SMD:R_0603_1608Metric, F.Cu at (188.0, 92.4)
- added R6: 0.01R, Resistor_SMD:R_Shunt_Vishay_WSR2_WSR3, F.Cu at (95.2, 26.8)
- added R7: 0.01R, Resistor_SMD:R_Shunt_Vishay_WSR2_WSR3, F.Cu at (95.7, 36.8)
- added R8: 0.01R, Resistor_SMD:R_Shunt_Vishay_WSR2_WSR3, F.Cu at (95.5, 46.5)
- added R9: 0.01R, Resistor_SMD:R_Shunt_Vishay_WSR2_WSR3, F.Cu at (95.6, 57.5)
- added SW1: SW_Push, Button_Switch_THT:SW_PUSH_1P1T_6x3.5mm_H5.0_APEM_MJTP1250, F.Cu at (132.1, 33.2)
- added U2: ~, Package_TO_SOT_SMD:SOT-23-5_HandSoldering, F.Cu at (105.5, 25.0)
- added U3: ~, Package_TO_SOT_SMD:SOT-23-5_HandSoldering, F.Cu at (107.0, 36.4)
- added U4: ~, Package_TO_SOT_SMD:SOT-23-5_HandSoldering, F.Cu at (108.7, 45.4)
- added U5: ~, Package_TO_SOT_SMD:SOT-23-5_HandSoldering, F.Cu at (106.5, 57.5)
- added U6: LM1117DT-3.3, Package_TO_SOT_SMD:TO-252-3_TabPin2, F.Cu at (133.1, 59.3)
- J1: footprint Connector_Wago:Wago_734-136_1x06_P3.50mm_Vertical -> Connector_PinHeader_1.00mm:PinHeader_1x06_P1.00mm_Vertical
- moved J1 101.2 mm to (187.3, 95.7), turned to -90 degrees
- moved U1 100.7 mm to (194.6, 64.9)
Connections:
- U1 pad 10: unconnected-(U1-IO25-Pad10) -> /CurrentSensing/INLine03
- U1 pad 12: unconnected-(U1-IO27-Pad12) -> /CurrentSensing/INLine04
- U1 pad 24: unconnected-(U1-IO2-Pad24) -> /CurrentSensing/INLine02
- U1 pad 25: unconnected-(U1-IO0-Pad25) -> /CurrentSensing/INLine01
- U1 pad 30: unconnected-(U1-IO18-Pad30) -> Net-(D2-K)
- U1 pad 6: unconnected-(U1-IO34-Pad6) -> /CurrentSensing/CurrLine03
- U1 pad 7: unconnected-(U1-IO35-Pad7) -> /CurrentSensing/CurrLine04
- U1 pad 8: unconnected-(U1-IO32-Pad8) -> /CurrentSensing/CurrLine01
- U1 pad 9: unconnected-(U1-IO33-Pad9) -> /CurrentSensing/CurrLine02
Other:
- board outline added: 50 x 50 mm
